File: IBM31SD.kicad_sch (KiCad schematic)
At the start: 93 parts, among them U1 7400, U2 7404, U3 MC1472

Commit message: Updated info on IBM part numbers
Parts:
- C? (x5): value 8.6uF -> 8.2uF 12V
- C?: value 4.2uF -> 3.9uF 20V
- C? (x7): IBM 1539475 -> 1589475
- C?: value 126pF -> 120pF
- C?: IBM 491 309 123 8210 -> 0491309
- C?: value 172pF -> 180pF
- C?: value 1uF (35V?) -> 0.68uF 50V
- RN?: value 120K -> 121K; IBM 2408834 -> 2408334
Other:
- note added: "INNER_TRACKS: ACTIVE FROM TRACK 43-76"
Changed lines of the file:
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@@
     (effects (font (size 1.27 1.27)) (justify left bottom))
   )
+  (text "INNER_TRACKS: ACTIVE \nFROM TRACK 43-76" (at 88.9 125.73 0)
+    (effects (font (size 1.27 1.27)) (justify left bottom))
+  )
   (label "WRITE{slash}ERASE_EN" (at 68.58 118.11 180)
     (effects (font (size 1.27 1.27)) (justify right bottom))
@@
       (effects (font (size 1.27 1.27)) (justify left))
     )
-    (property "Value" "8.6uF" (id 1) (at 55.88 82.1181 0)
+    (property "Value" "8.2uF 12V" (id 1) (at 55.88 82.1181 0)
       (effects (font (size 1.27 1.27)) (justify left))
     )
@@
       (effects (font (size 1.27 1.27)) (justify left))
     )
-    (property "Value" "4.2uF" (id 1) (at 220.98 266.2681 0)
+    (property "Value" "3.9uF 20V" (id 1) (at 220.98 266.2681 0)
       (effects (font (size 1.27 1.27)) (justify left))
     )
@@
       (effects (font (size 1.27 1.27)) (justify left))
     )
-    (property "Value" "8.6uF" (id 1) (at 208.28 71.9581 0)
+    (property "Value" "8.2uF 12V" (id 1) (at 208.28 71.9581 0)
       (effects (font (size 1.27 1.27)) (justify left))
     )
@@
       (effects (font (size 1.27 1.27)) hide)
     )
-    (property "IBM" "1539475" (id 4) (at 199.39 278.13 0)
+    (property "IBM" "1589475" (id 4) (at 199.39 278.13 0)
       (effects (font (size 1.27 1.27)) (justify left))
     )
@@
       (effects (font (size 1.27 1.27)) (justify left))
     )
-    (property "Value" "8.6uF" (id 1) (at 161.29 83.3881 0)
+    (property "Value" "8.2uF 12V" (id 1) (at 161.29 83.3881 0)
       (effects (font (size 1.27 1.27)) (justify left))
     )
@@
       (effects (font (size 1.27 1.27)) (justify left))
     )
-    (property "Value" "126pF" (id 1) (at 302.26 73.66 0)
+    (property "Value" "120pF" (id 1) (at 302.26 73.66 0)
       (effects (font (size 1.27 1.27)) (justify left))
     )
@@
       (effects (font (size 1.27 1.27)) hide)
     )
-    (property "IBM" "491 309 123 8210" (id 4) (at 251.46 93.98 90)
+    (property "IBM" "0491309" (id 4) (at 251.46 93.98 90)
       (effects (font (size 1.27 1.27)) (justify left))
     )
@@
       (effects (font (size 1.27 1.27)) hide)
     )
-    (property "IBM" "1539475" (id 4) (at 228.6 77.47 0)
+    (property "IBM" "1589475" (id 4) (at 228.6 77.47 0)
       (effects (font (size 1.27 1.27)) (justify left))
     )
@@
       (effects (font (size 1.27 1.27)) hide)
     )
-    (property "IBM" "1539475" (id 4) (at 247.65 77.47 0)
+    (property "IBM" "1589475" (id 4) (at 247.65 77.47 0)
       (effects (font (size 1.27 1.27)) (justify left))
     )
@@
       (effects (font (size 1.27 1.27)) (justify left))
     )
-    (property "Value" "172pF" (id 1) (at 161.29 68.58 0)
+    (property "Value" "180pF" (id 1) (at 161.29 68.58 0)
       (effects (font (size 1.27 1.27)) (justify left))
     )
@@
       (effects (font (size 1.27 1.27)) hide)
     )
-    (property "IBM" "1539475" (id 4) (at 341.63 87.63 0)
+    (property "IBM" "1589475" (id 4) (at 341.63 87.63 0)
       (effects (font (size 1.27 1.27)) (justify left))
     )
@@
       (effects (font (size 1.27 1.27)) hide)
     )
-    (property "IBM" "1539475" (id 4) (at 237.49 68.58 90)
+    (property "IBM" "1589475" (id 4) (at 237.49 68.58 90)
       (effects (font (size 1.27 1.27)) (justify left))
     )
@@
       (effects (font (size 1.27 1.27)) hide)
     )
-    (property "IBM" "1539475" (id 4) (at 236.22 55.88 90)
+    (property "IBM" "1589475" (id 4) (at 236.22 55.88 90)
       (effects (font (size 1.27 1.27)) (justify left))
     )
@@
       (effects (font (size 1.27 1.27)) (justify left))
     )
-    (property "Value" "8.6uF" (id 1) (at 69.85 82.1181 0)
+    (property "Value" "8.2uF 12V" (id 1) (at 69.85 82.1181 0)
       (effects (font (size 1.27 1.27)) (justify left))
     )
@@
       (effects (font (size 1.27 1.27)) (justify left))
     )
-    (property "Value" "1uF (35V?)" (id 1) (at 52.07 153.67 0)
+    (property "Value" "0.68uF 50V" (id 1) (at 52.07 153.67 0)
       (effects (font (size 1.27 1.27)) (justify left))
     )
@@
       (effects (font (size 1.27 1.27)) (justify left))
     )
-    (property "Value" "8.6uF" (id 1) (at 261.62 50.3681 0)
+    (property "Value" "8.2uF 12V" (id 1) (at 261.62 50.3681 0)
       (effects (font (size 1.27 1.27)) (justify left))
     )
@@
       (effects (font (size 1.27 1.27)) (justify left))
     )
-    (property "Value" "120K" (id 1) (at 308.61 44.4499 0)
+    (property "Value" "121K" (id 1) (at 308.61 44.4499 0)
       (effects (font (size 1.27 1.27)) (justify left))
     )
@@
       (effects (font (size 1.27 1.27)) hide)
     )
-    (property "IBM" "2408834" (id 4) (at 308.61 46.99 0)
+    (property "IBM" "2408334" (id 4) (at 308.61 46.99 0)
       (effects (font (size 1.27 1.27)) (justify left))
     )
@@
       (effects (font (size 1.27 1.27)) hide)
     )
-    (property "IBM" "1539475" (id 4) (at 59.69 54.61 0)
+    (property "IBM" "1589475" (id 4) (at 59.69 54.61 0)
       (effects (font (size 1.27 1.27)) (justify left))
     )
@@
     )
     (path "/14d6e43b-a1cd-4e22-99f8-ed8c64722a8d"
-      (reference "C?") (unit 1) (value "8.6uF") (footprint "")
+      (reference "C?") (unit 1) (value "8.2uF 12V") (footprint "")
     )
     (path "/1adc0b43-bd82-437a-af45-843656025739"
-      (reference "C?") (unit 1) (value "4.2uF") (footprint "")
+      (reference "C?") (unit 1) (value "3.9uF 20V") (footprint "")
     )
     (path "/2413c2cd-a7fb-4bbd-a37c-a29c4f149337"
-      (reference "C?") (unit 1) (value "8.6uF") (footprint "")
+      (reference "C?") (unit 1) (value "8.2uF 12V") (footprint "")
     )
     (path "/2c1f0993-2b7e-43f0-98c2-d3619960915b"
@@
     )
     (path "/33e5aa48-ff07-4966-b20d-77c822330528"
-      (reference "C?") (unit 1) (value "8.6uF") (footprint "")
+      (reference "C?") (unit 1) (value "8.2uF 12V") (footprint "")
     )
     (path "/3d536276-10a3-40b6-9dc8-702fc2345240"
-      (reference "C?") (unit 1) (value "126pF") (footprint "")
+      (reference "C?") (unit 1) (value "120pF") (footprint "")
     )
     (path "/4205bc9a-45de-4acf-8bbb-a6c78dd88708"
@@
     )
     (path "/5566ce26-169f-4936-b1f1-64839c7efcd5"
-      (reference "C?") (unit 1) (value "172pF") (footprint "")
+      (reference "C?") (unit 1) (value "180pF") (footprint "")
     )
     (path "/59e7f232-854d-4d2f-94e3-fbcc3a14e691"
@@
     )
     (path "/a49cd791-ba78-49f2-a34e-7bd9b8845274"
-      (reference "C?") (unit 1) (value "8.6uF") (footprint "")
+      (reference "C?") (unit 1) (value "8.2uF 12V") (footprint "")
     )
     (path "/a8577759-b537-4ba6-9ca9-7cbc6104577d"
-      (reference "C?") (unit 1) (value "1uF (35V?)") (footprint "")
+      (reference "C?") (unit 1) (value "0.68uF 50V") (footprint "")
     )
     (path "/c804b67e-cebf-47e1-b69b-87bc6aebc906"
-      (reference "C?") (unit 1) (value "8.6uF") (footprint "")
+      (reference "C?") (unit 1) (value "8.2uF 12V") (footprint "")
     )
     (path "/feb39efd-8410-444b-9b77-624ab79f87a8"
@@
     )
     (path "/e3b360cb-df06-4b60-a314-582320375827"
-      (reference "RN?") (unit 1) (value "120K") (footprint "Resistor_THT:R_Array_SIP4")
+      (reference "RN?") (unit 1) (value "121K") (footprint "Resistor_THT:R_Array_SIP4")
     )
     (path "/f25d7f0c-e846-42ba-9e00-2f092d1ab813"
